Commit message: add gripper as planning group

File: sawback_moveit_config/srdf/sawback.srdf.xacro (robot description, xacro)
@@ -11,8 +11,19 @@
     <!--SUBGROUPS: Groups can also be formed by referencing to already defined group names-->
     <group name="right_arm">
-        <chain base_link="base" tip_link="right_gripper_tip"/>
+      <chain base_link="base" tip_link="right_gripper_tip"/>
     </group>
+    <group name="hand">
+      <joint name="right_gripper_l_finger_joint"/>
+      <joint name="right_gripper_r_finger_joint"/>
+      <joint name="right_hand"/>
+    </group>
+    <group_state name="open" group="hand">
+      <joint name="right_gripper_l_finger_joint" value="0.0416" />
+    </group_state>
+    <group_state name="close" group="hand">
+      <joint name="right_gripper_l_finger_joint" value="0" />
+    </group_state>
     <!--END EFFECTOR: Purpose: Represent information about an end effector.-->
-    <end_effector name="right_hang_eef" parent_link="right_hand" group="right_arm"/>
+    <end_effector name="right_hang_eef" parent_link="right_hand" group="hand" parent_group="right_arm"/>
     <!--DISABLE COLLISIONS: By default it is assumed that any link of the robot could potentially come into collision with any other link in the robot. This tag disables collision checking between a specified pair of links. -->
     <disable_collisions link1="chassis_link" link2="controller_enclosure" reason="Adjacent"/>

Commit message: update

File: sawback_moveit_config/srdf/sawback.srdf.xacro (robot description, xacro)
@@ -16,11 +16,13 @@
       <joint name="right_gripper_l_finger_joint"/>
       <joint name="right_gripper_r_finger_joint"/>
-      <joint name="right_hand"/>
+      <!-- <joint name="right_hand"/> -->
     </group>
     <group_state name="open" group="hand">
       <joint name="right_gripper_l_finger_joint" value="0.0416" />
+      <!-- <joint name="right_gripper_r_finger_joint" value="0.0416" /> -->
     </group_state>
     <group_state name="close" group="hand">
-      <joint name="right_gripper_l_finger_joint" value="0" />
+      <joint name="right_gripper_l_finger_joint" value="0.0" />
+      <!-- <joint name="right_gripper_r_finger_joint" value="0.0" /> -->
     </group_state>
     <!--END EFFECTOR: Purpose: Represent information about an end effector.-->

Commit message: add ready state to right_arm group

File: sawback_moveit_config/srdf/sawback.srdf.xacro (robot description, xacro)
@@ -13,4 +13,13 @@
       <chain base_link="base" tip_link="right_gripper_tip"/>
     </group>
+    <group_state name="ready" group="right_arm">
+      <joint name="right_j0" value="0.136716796875"/>
+      <joint name="right_j1" value="-1.345919921875"/>
+      <joint name="right_j2" value="-0.3328642578125"/>
+      <joint name="right_j3" value="2.0867880859375"/>
+      <joint name="right_j4" value="-0.19401171875"/>
+      <joint name="right_j5" value="-0.8204111328125"/>
+      <joint name="right_j6" value="-1.0447021484375"/>
+    </group_state>
     <group name="hand">
       <joint name="right_gripper_l_finger_joint"/>
